Commit message: urdf *2, *3 joint 범위 변경

File: glove_based/assets/v6_right/v6_right.bk.urdf (robot description, URDF)
Before this commit: robot v6_right, 22 links, 21 joints
Joints:
- joint joint_02: limit lower=-0.087266 upper=1.5708 effort=0.38 velocity=8.70 -> lower=-1.5708 upper=1.5708 effort=0.38 velocity=8.70
- joint joint_03: limit lower=-0.087266 upper=1.5708 effort=0.38 velocity=8.70 -> lower=-1.5708 upper=1.5708 effort=0.38 velocity=8.70
- joint joint_12: limit lower=-0.087266 upper=1.5708 effort=0.38 velocity=8.70 -> lower=-1.5708 upper=1.5708 effort=0.38 velocity=8.70
- joint joint_13: limit lower=-0.087266 upper=1.5708 effort=0.38 velocity=8.70 -> lower=-1.5708 upper=1.5708 effort=0.38 velocity=8.70
- joint joint_22: limit lower=-0.087266 upper=1.5708 effort=0.38 velocity=8.70 -> lower=-1.5708 upper=1.5708 effort=0.38 velocity=8.70
- joint joint_23: limit lower=-0.087266 upper=1.5708 effort=0.38 velocity=8.70 -> lower=-1.5708 upper=1.5708 effort=0.38 velocity=8.70
- joint joint_32: limit lower=-0.087266 upper=1.5708 effort=0.38 velocity=8.70 -> lower=-1.5708 upper=1.5708 effort=0.38 velocity=8.70
- joint joint_33: limit lower=-0.087266 upper=1.5708 effort=0.38 velocity=8.70 -> lower=-1.5708 upper=1.5708 effort=0.38 velocity=8.70
- joint joint_42: limit lower=-0.087266 upper=1.5708 effort=0.38 velocity=8.70 -> lower=-1.5708 upper=1.5708 effort=0.38 velocity=8.70
- joint joint_43: limit lower=-0.087266 upper=1.5708 effort=0.38 velocity=8.70 -> lower=-1.5708 upper=1.5708 effort=0.38 velocity=8.70
