Commit message: Test aph

File: glove_based/assets/aph_right/aph_right.urdf (robot description, URDF)
Before this commit: robot aph_right, 21 links, 20 joints
Links:
- added link virtual_base
Joints:
- added joint virtual_base_to_base_link: type fixed, parent virtual_base, child base_link, origin xyz=-0.00125 0 -0.0905 rpy=0 0 1.5708
